Commit message: Latitude and longitude as parameter of the xacro file.

File: urdf/base_gazebo.xacro (robot description, xacro)
@@ -26,5 +26,5 @@
   <!-- Optional sensor plugins - called by macros defined above -->
   <xacro:if value="$(arg gps)">
-    <xacro:kingfisher_gps_gazebo name="kingfisher"/>
+    <xacro:kingfisher_gps_gazebo name="kingfisher" latitude="$(arg latitude)" longitude="$(arg longitude)"/>
   </xacro:if>
   <xacro:if value="$(arg imu)">

File: urdf/gps_gazebo.xacro (robot description, xacro)
@@ -1,5 +1,5 @@
 <?xml version="1.0"?>
 <robot xmlns:xacro="http://ros.org/wiki/xacro">
-  <xacro:macro name="kingfisher_gps_gazebo" params="name">
+  <xacro:macro name="kingfisher_gps_gazebo" params="name latitude longitude">
     <gazebo>
       <plugin name="gps_plugin_${name}" filename="libhector_gazebo_ros_gps.so">
@@ -8,8 +8,8 @@
 	<bodyName>base_link</bodyName>
 	<frameId>base_link</frameId>
-	<topicName>gps/fix</topicName>
+	<topicName>navsat/fix</topicName>
 	<velocityTopicName>fix_velocity</velocityTopicName>
-	<referenceLatitude>36.6</referenceLatitude>
-	<referenceLongitude>-121.9</referenceLongitude>
+	<referenceLatitude>${latitude}</referenceLatitude>
+	<referenceLongitude>${longitude}</referenceLongitude>
 	<referenceAltitude>10.0</referenceAltitude>
 	<offset>0.0 0.0 0.0</offset>
